File: rev4/hardware/step400_proto_r4.sch (EAGLE design)
At the start: 208 parts, among them IC1 0982_W5500LONG, J2 SDCARD_SLOT_TF-115K, J3 691321300004, J4 691321300004, J5 691321300004, J6 691321300004, Q1 SUD50P08-25L-E3, Q2 32.768kHz, Q3 16MHz, U1 USBLC6-2SC6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

Commit message: Added the schematics PDF, updated the Max example patch.
Other:
- note added: "r4 memo"
- note added: "updated components - screw terminal - connector XA + 3.81mm - microSD card slot - limit SW - 3.3V regulator"
- note removed: "Prototype r3 for TASKO"
- note removed: "update components - screw terminal - connector XA + 3.81mm - microSD card slot - limit SW - 3.3V regulator"
Changed lines of the file:
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@@
 <?xml version="1.0" encoding="utf-8"?>
 <!DOCTYPE eagle SYSTEM "eagle.dtd">
-<eagle version="9.6.0">
+<eagle version="9.6.2">
 <drawing>
 <settings>
@@
 <text x="241.3" y="182.88" size="1.778" layer="97" align="center-left">SCL</text>
 <text x="243.84" y="154.94" size="1.778" layer="97" align="center-left">D31</text>
-<text x="12.7" y="40.64" size="1.778" layer="97">Prototype r3 for TASKO</text>
-<text x="12.7" y="35.56" size="1.778" layer="97" align="top-left">update components
+<text x="12.7" y="40.64" size="1.778" layer="97">r4 memo</text>
+<text x="12.7" y="35.56" size="1.778" layer="97" align="top-left">updated components
 - screw terminal
 - connector XA + 3.81mm
